File: led-music-pulse/Schematic/musicpulse.brd (EAGLE design)
At the start: 70.8 x 48.2 mm, 13 parts

Commit message: Added schematic
Parts:
- removed C1: 10uF, SparkFun-Capacitors:CPOL-RADIAL-2.5MM-5MM
- removed POT: (no value), SparkFun-Connectors:1X02
- removed U$1: TEENSY_3.5/3.6, Teensy356:TEENSY_3.5/3.6
- added C2: 0.1uF, BeagleBone_Black_Wireless:C1206
- added C3: 0.33uF, BeagleBone_Black_Wireless:C1206
- added C4: 10uF, BeagleBone_Black_Wireless:C1206
- added D1: GREEN, SparkFun-LED:LED-1206
- added D2: Yellow, SparkFun-LED:LED-1206
- added IC1: UA78M33DCY, linear:SOT223
- added POT1, POT2: (no value), SparkFun-Connectors:1X03
- added U$2: TEENSY_3.1-3.2_DIL+4, Teensy_3_and_LC_Series_Boards_v1.4:TEENSY_3.0-3.2&LC_DIL+4
- R1, R2, R3: device SparkFun-Resistors:AXIAL-0.3 -> BeagleBone_Black_Wireless:R1206
- R4, R5: value 10k -> 100; device SparkFun-Resistors:AXIAL-0.3 -> BeagleBone_Black_Wireless:R1206
- moved R5 105.1 mm to (-27.9, -62.2), turned to 0 degrees
- moved R4 104.4 mm to (-27.9, -55.9), turned to 0 degrees
- moved R1 84.7 mm to (-8.89, -41.9), turned to 0 degrees
- moved R3 63.9 mm to (-8.89, -35.6)
- moved R2 46.6 mm to (-8.89, -29.2)
Connections:
- removed net POT: POT.2, U$1.8
- removed net SLIDE1: R5.P$2, U$1.9/CS
- removed net SLIDE2: R4.P$2, U$1.10/CS
- new net 3.3V: U$2.3.3V
- new net AGND: U$2.AGND
- new net AREF: U$2.AREF
- new net LED_GREEN: C3.1, IC1.3, R4.1
- new net LED_YELLOW: R5.2, U$2.10
- new net N$2: D1.A, R4.2
- new net POT1: POT1.2, U$2.15/A1
- new net POT2: POT2.2, U$2.16/A2
- new net SLIDE: SLIDER.2, U$2.12
- new net VUSB: U$2.VUSB
- net AUDIO_IN: now also C4.1, R2.2, R3.1, U$2.14/A0; no longer C1.2, R2.P$2, R3.P$1, U$1.5
- net GND: now also C2.2, C3.2, D1.C, D2.C, IC1.2, IC1.4, POT1.3, POT2.3, PWR.1, R2.1, SLIDER.1, U$2.GND; no longer PWR.2, R2.P$1, U$1.GND
- net LIGHTS: now also U$2.9; no longer U$1.7
- net N$1: now also C2.1, IC1.1, PWR.2; no longer PUSH.1, R1.P$1
- net N$3: now also R1.2; no longer R5.P$1, SLIDER.1
- net N$4: now also D2.A, R5.1; no longer R4.P$1, SLIDER.3
- net N$5: now also C4.2; no longer C1.1
- net PUSH: now also PUSH.1, R1.1, U$2.11; no longer R1.P$2, U$1.6
- net VCC: now also POT1.1, POT2.1, R3.2, SLIDER.3, U$2.VIN; no longer POT.1, PWR.1, R3.P$2, SLIDER.2, U$1.VIN
Routing:
- net VCC: track 84.0 -> 3.81 mm
- net PUSH: track 36.3 -> 0.00 mm
- net AUDIO_IN: track 26.6 -> 0.00 mm
- net POT: track 23.3 -> 0.00 mm
- net SLIDE2: track 18.4 -> 0.00 mm
- net SLIDE1: track 15.9 -> 0.00 mm
- net N$5: track 9.02 -> 0.00 mm
- net LIGHTS: track 20.6 -> 12.4 mm
- net N$4: track 3.81 -> 0.00 mm
- net N$3: track 3.81 -> 0.00 mm
- net N$1: track 3.81 -> 0.00 mm
