File: led-music-pulse/Schematic/musicpulse.sch (EAGLE design)
At the start: 13 parts

Commit message: Added schematic
Parts:
- removed C1: 10uF, SparkFun-Capacitors:10UF-POLAR-RADIAL-2.5MM-25V-20%
- removed POT: (no value), SparkFun-Connectors:CONN_02
- removed U$1: TEENSY_3.5/3.6, Teensy356:TEENSY_3.5/3.6
- added C2: 0.1uF, BeagleBone_Black_Wireless:C-USC1206
- added C3: 0.33uF, BeagleBone_Black_Wireless:C-USC1206
- added C4: 10uF, BeagleBone_Black_Wireless:C-USC1206
- added D1: GREEN, SparkFun-LED:LED-GREEN1206
- added D2: Yellow, SparkFun-LED:LED-YELLOWLILYPAD
- added IC1: UA78M33DCY, linear:UA78M33DCY
- added POT1, POT2: (no value), SparkFun-Connectors:CONN_03
- added U$2: TEENSY_3.1-3.2_DIL+4, Teensy_3_and_LC_Series_Boards_v1.4:TEENSY_3.1-3.2_DIL+4
- R1, R2, R3: device SparkFun-Resistors:10KOHM-HORIZ-1/4W-1% -> BeagleBone_Black_Wireless:R-US_R1206
- R4, R5: value 10k -> 100; device SparkFun-Resistors:10KOHM-HORIZ-1/4W-1% -> BeagleBone_Black_Wireless:R-US_R1206
Connections:
- removed net POT: POT.2, U$1.8
- removed net SLIDE1: R5.2, U$1.9/CS
- removed net SLIDE2: R4.2, U$1.10/CS
- new net LED_GREEN: C3.1, IC1.VO, R4.1
- new net LED_YELLOW: R5.2, U$2.10/TX2/PWM
- new net N$2: D1.A, R4.2
- new net POT1: POT1.2, U$2.15/A1/T
- new net POT2: POT2.2, U$2.16/A2/T
- new net SLIDE: SLIDER.2, U$2.12/MISO
- net AUDIO_IN: now also C4.1, U$2.14/A0; no longer C1.-, U$1.5
- net GND: now also C2.2, C3.2, D1.C, D2.C, IC1.GND, IC1.GND@1, POT1.3, POT2.3, PWR.1, SLIDER.1, U$2.GND; no longer PWR.2, U$1.GND
- net LIGHTS: now also U$2.9/RX2/PWM; no longer U$1.7
- net N$1: now also C2.1, IC1.VI, PWR.2; no longer PUSH.1, R1.1
- net N$3: now also R1.2; no longer R5.1, SLIDER.1
- net N$4: now also D2.A, R5.1; no longer R4.1, SLIDER.3
- net N$5: now also C4.2; no longer C1.+
- net PUSH: now also PUSH.1, R1.1, U$2.11/MOSI; no longer R1.2, U$1.6
- net VCC: now also POT1.1, POT2.1, SLIDER.3, U$2.VIN; no longer POT.1, PWR.1, SLIDER.2, U$1.VIN
Other:
- moved on the sheet: LIGHTS, PUSH, PWR, R1, R4, R5, SLIDER
